Commit message: general commit

File: artificial_hands_description/urdf/robotiq_ft300.urdf.xacro (robot description, xacro)
@@ -30,5 +30,5 @@
                 <origin xyz="0 0 0" rpy="0 0 0" />
                 <geometry>
-                    <mesh filename="package://robotiq_ft_sensor/meshes/visual/robotiq_ft300.STL"/>
+                    <mesh filename="package://artificial_hands_description/meshes/visual/robotiq_ft300.STL"/>
                 </geometry>
                 <material name="Robotiq-Black">
@@ -39,5 +39,5 @@
                 <origin xyz="0 0 0" rpy="0 0 0" />
                 <geometry>
-                    <mesh filename="package://robotiq_ft_sensor/meshes/collision/robotiq_ft300.STL"/>
+                    <mesh filename="package://artificial_hands_description/meshes/collision/robotiq_ft300.STL"/>
                 </geometry>
             </collision>
@@ -48,5 +48,5 @@
                 <origin xyz="0 0 0" rpy="0 0 0" />
                 <geometry>
-                    <mesh filename="package://robotiq_ft_sensor/meshes/visual/mountings/robotiq_ft300-G-062-COUPLING_G-50-4M6-1D6_20181119.STL"/>
+                    <mesh filename="package://artificial_hands_description/meshes/visual/mountings/robotiq_ft300-G-062-COUPLING_G-50-4M6-1D6_20181119.STL"/>
                 </geometry>
                 <material name="Robotiq-Grey">
