Commit message: restored default from moveit_setup_assistant

File: artificial_hands_description/urdf/arm_base.urdf.xacro (robot description, xacro)
@@ -22,5 +22,5 @@
       <origin xyz="0 0 0.3" rpy="0 0 0"/>
       <geometry>
-        <box size="0.2 0.2 0.55"/>
+        <box size="0.2 0.2 0.6"/>
       </geometry>
     </collision>

File: artificial_hands_description/urdf/mia_hand_on_ur5.urdf.xacro (robot description, xacro)
@@ -1,4 +1,4 @@
 <?xml version="1.0"?>
-<robot xmlns:xacro="http://wiki.ros.org/xacro" name="mia_hand_on_ur5_robot_gazebo">
+<robot xmlns:xacro="http://wiki.ros.org/xacro" name="mia_hand_on_ur5">
   <!-- Make use of UR5 macro -->
   <xacro:include filename="$(find ur_description)/urdf/inc/ur5_macro.xacro" />
