Commit message: fixed position of sensor_frame

File: artificial_hands_description/urdf/onrobot_hex_e.urdf.xacro (robot description, xacro)
@@ -31,6 +31,6 @@
   <link name="hex_sensor_frame"/>
   <joint name="hex_sensor_joint" type="fixed">
-    <origin xyz="0 0 0.016" rpy="0 0 0" />
-    <parent link="hex_mounting_plate" />
+    <origin xyz="0 0 0" rpy="0 0 0" />
+    <parent link="hex_ee_mounting_plate" />
     <child link="hex_sensor_frame" />
   </joint>
