Commit message: commited minor changes

File: artificial_hands_description/urdf/mia_hand_on_ur10e.urdf.xacro (robot description, xacro)
@@ -1,8 +1,9 @@
 <?xml version="1.0"?>
-<robot xmlns:xacro="http://wiki.ros.org/xacro" name="mia_hand_on_ur5">
-  <!-- Make use of UR macro -->
-  <xacro:include filename="$(find ur_description)/urdf/inc/ur_macro.xacro"/>
+<robot xmlns:xacro="http://wiki.ros.org/xacro" name="mia_hand_on_ur10e">
+  <!-- Make use of UR10e macro -->
+  <xacro:include filename="$(find ur_description)/urdf/inc/ur10e_macro.xacro"/>
   <!-- Instantiate the UR robot and pass it all the required arguments. -->
-  <xacro:ur_robot
+  <xacro:ur10e_robot
+    prefix=""
   />
   <!-- Arm base -->

File: artificial_hands_description/urdf/mia_hand_on_ur5.urdf.xacro (robot description, xacro)
@@ -1,17 +1,9 @@
 <?xml version="1.0"?>
-<robot xmlns:xacro="http://wiki.ros.org/xacro" name="mia_hand_on_ur">
-  <!-- Make use of UR macro -->
-  <xacro:include filename="$(find ur_description)/urdf/inc/ur_macro.xacro"/>
+<robot xmlns:xacro="http://wiki.ros.org/xacro" name="mia_hand_on_ur5">
+  <!-- Make use of UR5 macro -->
+  <xacro:include filename="$(find ur_description)/urdf/inc/ur5_macro.xacro"/>
   <!-- Instantiate the UR robot and pass it all the required arguments. -->
-  <xacro:ur_robot
+  <xacro:ur5_robot
     prefix=""
-    joint_limits_parameters_file="$(arg joint_limit_params)"
-    kinematics_parameters_file="$(arg kinematics_params)"
-    physical_parameters_file="$(arg physical_params)"
-    visual_parameters_file="$(arg visual_params)"
-    transmission_hw_interface="$(arg transmission_hw_interface)"
-    safety_limits="$(arg safety_limits)"
-    safety_pos_margin="$(arg safety_pos_margin)"
-    safety_k_position="$(arg safety_k_position)"
   />
   <!-- Arm base -->

File: artificial_hands_description/urdf/onrobot_hex_e.urdf.xacro (robot description, xacro)
@@ -23,20 +23,20 @@
     </collision>
   </link>
+  <gazebo reference="hex_mounting_plate">
+    <selfCollide>false</selfCollide>
+  </gazebo>
+  <link name="hex_sensor_frame"/>
+  <joint name="hex_sensor_joint" type="fixed">
+    <origin xyz="0 0 0.037" rpy="0 0 0" />
+    <parent link="hex_mounting_plate" />
+    <child link="hex_sensor_frame" />
+  </joint>
   <link name="hex_ee_mounting_plate"/>
   <joint name="hex_ee_mounting_joint" type="fixed">
-    <origin xyz="0 0 0.037" rpy="0 0 0" />
-    <parent link="hex_mounting_plate" />
+    <origin xyz="0 0 0" rpy="0 0 0" />
+    <parent link="hex_sensor_frame" />
     <child link="hex_ee_mounting_plate" />
   </joint>
-  <link name="hex_sensor_frame"/>
-  <joint name="hex_sensor_joint" type="fixed">
-    <origin xyz="0 0 0" rpy="0 0 0" />
-    <parent link="hex_ee_mounting_plate" />
-    <child link="hex_sensor_frame" />
-  </joint>
-  <gazebo reference="hex_mounting_plate">
-    <selfCollide>False</selfCollide>
-  </gazebo>
-    <!-- Enable joint feedback representing the ft_sensor-->
+  <!-- Enable joint feedback representing the ft_sensor-->
   <gazebo reference="hex_sensor_joint">
     <preserveFixedJoint>true</preserveFixedJoint>
@@ -47,5 +47,5 @@
     <plugin name="gazebo_ft_sensor" filename="libgazebo_ros_ft_sensor.so">
       <updateRate>500.0</updateRate>
-        <topicName>hex_ft_sensor</topicName>
+        <topicName>gazebo/ft_sensor</topicName>
         <!-- <gaussianNoise>0.0</gaussianNoise> -->
         <jointName>hex_sensor_joint</jointName>
