Commit message: replaced robotiq_ft_frame with a new ft_sensor_frame

File: artificial_hands_description/urdf/inc/mia_hand_on_ur5.xacro (robot description, xacro)
@@ -29,4 +29,11 @@
       <origin xyz="0 0 -0.004" rpy="0 0 -${pi/2}"/>
   </xacro:robotiq_ft300>
+  <!-- Move the sensor frame according to the real hw -->
+  <link name="ft_sensor_frame"/>
+  <joint name="ft_frame_joint" type="fixed">
+    <origin xyz="0 0 0" rpy="0 0 0"/>
+    <parent link="robotiq_ft_frame_id"/>
+    <child link="ft_sensor_frame"/>
+  </joint>
   <!-- Enable joint feedback representing the ft_sensor-->
   <gazebo reference="measurment_joint">
@@ -71,8 +78,8 @@
     <selfCollide>False</selfCollide>
   </gazebo>
-  <!-- Make connection between robotiq_ft_sensor and mia hand -->
+  <!-- Make connection between ft_sensor_frame and mia hand -->
   <joint name="mia_fix" type="fixed">
     <origin xyz="0 0 0.022" rpy="${pi/2} 0 ${pi/2}"/>
-    <parent link="robotiq_ft_frame_id"/>
+    <parent link="ft_sensor_frame"/>
     <child link="palm"/>
   </joint>

File: artificial_hands_description/urdf/mia_hand_on_ur5.urdf.xacro (robot description, xacro)
@@ -19,4 +19,11 @@
       <origin xyz="0 0 -0.004" rpy="0 0 -${pi/2}"/>
   </xacro:robotiq_ft300>
+  <!-- Move the sensor frame according to the real hw -->
+  <link name="ft_sensor_frame"/>
+  <joint name="ft_frame_joint" type="fixed">
+    <origin xyz="0 0 0" rpy="0 0 0"/>
+    <parent link="robotiq_ft_frame_id"/>
+    <child link="ft_sensor_frame"/>
+  </joint>
   <!-- Enable joint feedback representing the ft_sensor-->
   <gazebo reference="measurment_joint">
@@ -61,8 +68,8 @@
     <selfCollide>False</selfCollide>
   </gazebo>
-  <!-- Make connection between robotiq_ft_sensor and mia hand -->
+  <!-- Make connection between ft_sensor_frame and mia hand -->
   <joint name="mia_fix" type="fixed">
     <origin xyz="0 0 0.022" rpy="${pi/2} 0 ${pi/2}"/>
-    <parent link="robotiq_ft_frame_id"/>
+    <parent link="ft_sensor_frame"/>
     <child link="palm"/>
   </joint>

Commit message: update toolkit with a new servo commander

File: artificial_hands_description/urdf/inc/mia_hand_on_ur5.xacro (robot description, xacro)
@@ -78,8 +78,8 @@
     <selfCollide>False</selfCollide>
   </gazebo>
-  <!-- Make connection between ft_sensor_frame and mia hand -->
+  <!-- Make connection between robotiq_ft_sensor and mia hand -->
   <joint name="mia_fix" type="fixed">
     <origin xyz="0 0 0.022" rpy="${pi/2} 0 ${pi/2}"/>
-    <parent link="ft_sensor_frame"/>
+    <parent link="robotiq_ft_frame_id"/>
     <child link="palm"/>
   </joint>

File: artificial_hands_description/urdf/mia_hand_on_ur5.urdf.xacro (robot description, xacro)
@@ -68,8 +68,8 @@
     <selfCollide>False</selfCollide>
   </gazebo>
-  <!-- Make connection between ft_sensor_frame and mia hand -->
+  <!-- Make connection between robotiq_ft_sensor and mia hand -->
   <joint name="mia_fix" type="fixed">
     <origin xyz="0 0 0.022" rpy="${pi/2} 0 ${pi/2}"/>
-    <parent link="ft_sensor_frame"/>
+    <parent link="robotiq_ft_frame_id"/>
     <child link="palm"/>
   </joint>

Commit message: fixed some warning in descriptions

File: artificial_hands_description/urdf/inc/mia_hand_on_ur5.xacro (robot description, xacro)
@@ -65,4 +65,11 @@
       <material name="DEFAULT_MTL.001"/>
     </visual>
+    <collision name="UR_flange">
+      <origin xyz="-0.023781363 -0.039999999 0.03784062" rpy="2.879793167 -1.3e-08 1.570796371"/>
+      <geometry>
+        <mesh filename="package://mia_hand_description/meshes/stl/1.001.stl" scale="0.000999987 0.000999987 0.000999987"/>
+      </geometry>
+      <material name="DEFAULT_MTL.001"/>
+    </collision>
   </link>
   <joint name="j_URflange" type="fixed">

File: artificial_hands_description/urdf/mia_hand_on_ur5.urdf.xacro (robot description, xacro)
@@ -55,4 +55,11 @@
       <material name="DEFAULT_MTL.001"/>
     </visual>
+    <collision name="UR_flange">
+      <origin xyz="-0.023781363 -0.039999999 0.03784062" rpy="2.879793167 -1.3e-08 1.570796371"/>
+      <geometry>
+        <mesh filename="package://mia_hand_description/meshes/stl/1.001.stl" scale="0.000999987 0.000999987 0.000999987"/>
+      </geometry>
+      <material name="DEFAULT_MTL.001"/>
+    </collision>
   </link>
   <joint name="j_URflange" type="fixed">

File: artificial_hands_description/urdf/robotiq_ft300.urdf.xacro (robot description, xacro)
@@ -54,10 +54,10 @@
                 </material>
             </visual>
-            <!-- <collision>
+            <collision>
                 <origin xyz="0 0 0" rpy="0 0 0" />
                 <geometry>
-                    <mesh filename="package://robotiq_ft_sensor/meshes/collision/mountings/robotiq_ft300-G-062-COUPLING_G-50-4M6-1D6_20181119.STL"/>
+                    <mesh filename="package://artificial_hands_description/meshes/collision/mountings/robotiq_ft300-G-062-COUPLING_G-50-4M6-1D6_20181119.STL"/>
                 </geometry>
-            </collision> -->
+            </collision>
         </link>
          <!-- Connect force sensor with mounting/coupling plate -->

Commit message: created pkg artificial_hands_nodes

File: artificial_hands_description/urdf/inc/mia_hand_on_ur5.xacro (robot description, xacro)
@@ -32,8 +32,44 @@
   <link name="ft_sensor_frame"/>
   <joint name="ft_frame_joint" type="fixed">
-    <origin xyz="0 0 0" rpy="0 0 0"/>
-    <parent link="robotiq_ft_frame_id"/>
+    <origin xyz="0 0 0.016" rpy="0 0 0"/>
+    <parent link="tool0"/>
     <child link="ft_sensor_frame"/>
   </joint>
+  <!-- OnRobot HEX-E v2-->
+  <!-- <link name="hex_mounting_plate">
+    <visual>
+      <origin xyz="0 0 0" rpy="0 0 0" />
+      <geometry>
+          <mesh filename="package://artificial_hands_description/meshes/visual/onrobot_hex_e.stl"/>
+      </geometry>
+      <material name="onrobot-grey">
+          <color rgba="0.4 0.4 0.4 1.0"/>
+      </material>
+    </visual>
+    <collision>
+      <origin xyz="0 0 0" rpy="0 0 0" />
+      <geometry>
+          <mesh filename="package://artificial_hands_description/meshes/collision/onrobot_hex_e.stl"/>
+      </geometry>
+    </collision>
+  </link>
+  <link name="hex_ee_mounting_plate"/>
+  <joint name="hex_mounting_joint" type="fixed">
+    <origin xyz="0 0 0.037" rpy="0 0 0" />
+    <parent link="hex_mounting_plate" />
+    <child link="hex_ee_mounting_plate" />
+  </joint>
+  <link name="hex_sensor_frame"/>
+  <joint name="hex_sensor_joint" type="fixed">
+    <origin xyz="0 0 0.037" rpy="0 0 0" />
+    <parent link="hex_mounting_plate" />
+    <child link="hex_sensor_frame" />
+  </joint> -->
+  <!-- Attach HEX sensor -->
+  <!-- <joint name="hex_fix" type="fixed">
+      <origin xyz="0 0 0.016" rpy="0 0 0"/>
+      <parent link="tool0" />
+      <child link="hex_mounting_plate" />
+  </joint> -->
   <!-- Enable joint feedback representing the ft_sensor-->
   <gazebo reference="measurment_joint">
