Commit message: created mia_hand_on_ur10 moveit config

File: artificial_hands_description/urdf/inc/mia_hand_on_ur.urdf.xacro (robot description, xacro)
@@ -1,8 +1,8 @@
 <?xml version="1.0"?>
-<robot xmlns:xacro="http://wiki.ros.org/xacro" name="mia_hand_on_ur10e">
-  <!-- Make use of UR5 macro -->
-  <xacro:include filename="$(find ur_description)/urdf/inc/ur10e_macro.xacro" />
-  <!-- Instantiate the UR5 Gazebo robot and pass it all the required arguments. -->
-  <xacro:ur10e_robot
+<robot xmlns:xacro="http://wiki.ros.org/xacro" name="mia_hand_on_ur">
+  <!-- Make use of UR macro -->
+  <xacro:include filename="$(find ur_description)/urdf/inc/ur_macro.xacro"/>
+  <!-- Instantiate the UR robot and pass it all the required arguments. -->
+  <xacro:ur_robot
     prefix=""
     joint_limits_parameters_file="$(arg joint_limit_params)"
@@ -15,5 +15,5 @@
     safety_k_position="$(arg safety_k_position)"
   />
-  <!-- Arm base (orange block representing mount for ur5 or ur10 arm) -->
+  <!-- Arm base -->
   <xacro:include filename="$(find artificial_hands_description)/urdf/arm_base.urdf.xacro" />
   <!-- Attach arm to the arm base -->
@@ -31,18 +31,4 @@
       <child link="hex_mounting_plate" />
   </joint>
-  <!-- Enable joint feedback representing the ft_sensor-->
-  <gazebo reference="hex_sensor_joint">
-    <preserveFixedJoint>true</preserveFixedJoint>
-    <provideFeedback>true</provideFeedback>
-  </gazebo>
-  <!-- The ft_sensor plugin -->
-  <gazebo>
-    <plugin name="gazebo_ft_sensor" filename="libgazebo_ros_ft_sensor.so">
-      <updateRate>500.0</updateRate>
-        <topicName>gazebo_ft_sensor</topicName>
-        <gaussianNoise>0.0</gaussianNoise>
-        <jointName>hex_sensor_joint</jointName>
-    </plugin>
-  </gazebo>
   <!-- Mia hand on UR flange -->
   <xacro:include filename="$(find artificial_hands_description)/urdf/mia_hand_on_ur_flange.urdf.xacro" />
@@ -54,13 +40,8 @@
   </joint>
   <!-- Instantiate the Mia hand Gazebo robot and pass it all the required arguments. -->
-  <!-- <xacro:include filename="$(find mia_hand_description)/urdf/mia_hand_gazebo.urdf.xacro" />
+  <xacro:include filename="$(find mia_hand_description)/urdf/mia_hand_gazebo.urdf.xacro" />
   <xacro:arg name="mia_hw_interface" default="Position" />
-  <xacro:mia_gazebo hw_interface_thumb_fle="$(arg mia_hw_interface)JointInterface"
-                    hw_interface_index_fle="$(arg mia_hw_interface)JointInterface"
-                    hw_interface_mrl_fle="$(arg mia_hw_interface)JointInterface"
-                    robotNamespace="" /> -->
-  <gazebo>
-    <plugin name="gazebo_ros_control" filename="libgazebo_ros_control.so">
-    </plugin>
-  </gazebo>
+  <xacro:mia_gazebo
+    robotNamespace=""
+  />
 </robot>

File: artificial_hands_description/urdf/mia_hand_on_ur10e.urdf.xacro (robot description, xacro)
@@ -1,8 +1,8 @@
 <?xml version="1.0"?>
-<robot xmlns:xacro="http://wiki.ros.org/xacro" name="mia_hand_on_ur5">
+<robot xmlns:xacro="http://wiki.ros.org/xacro" name="mia_hand_on_ur10e">
   <!-- Make use of UR macro -->
-  <xacro:include filename="$(find ur_description)/urdf/inc/ur5_macro.xacro"/>
+  <xacro:include filename="$(find ur_description)/urdf/inc/ur10e_macro.xacro"/>
   <!-- Instantiate the UR robot and pass it all the required arguments. -->
-  <xacro:ur5_robot
+  <xacro:ur10e_robot
     prefix=""
   />

File: artificial_hands_description/urdf/onrobot_hex_e.urdf.xacro (robot description, xacro)
@@ -2,4 +2,9 @@
 <robot xmlns:xacro="http://wiki.ros.org/xacro" name="onrobot_hex">
   <link name="hex_mounting_plate">
+    <inertial>
+      <origin xyz="0 0 0.016" rpy="-${pi/2} 0 0"/>
+      <mass value="0.245"/>
+      <inertia ixx="${99 / 1000000}" ixy="0" ixz="0" iyy="${142 / 1000000}" iyx="0" iyz="${-0.2 / 1000000}" izz="${99 / 1000000}" izx="0" izy="${-0.2 / 1000000}"/>
+    </inertial>
     <visual>
       <origin xyz="0 0 0.016" rpy="-${pi/2} 0 0" />
@@ -12,5 +17,5 @@
     </visual>
     <collision>
-      <origin xyz="0 0 0" rpy="0 0 0" />
+      <origin xyz="0 0 0.016" rpy="-${pi/2} 0 0" />
       <geometry>
           <mesh filename="package://artificial_hands_description/meshes/collision/onrobot_hex_e.stl"/>
@@ -30,3 +35,20 @@
     <child link="hex_sensor_frame" />
   </joint>
+  <gazebo reference="hex_mounting_plate">
+    <selfCollide>False</selfCollide>
+  </gazebo>
+    <!-- Enable joint feedback representing the ft_sensor-->
+  <gazebo reference="hex_sensor_joint">
+    <preserveFixedJoint>true</preserveFixedJoint>
+    <provideFeedback>true</provideFeedback>
+  </gazebo>
+  <!-- The ft_sensor plugin -->
+  <gazebo>
+    <plugin name="gazebo_ft_sensor" filename="libgazebo_ros_ft_sensor.so">
+      <updateRate>500.0</updateRate>
+        <topicName>hex_ft_sensor</topicName>
+        <!-- <gaussianNoise>0.0</gaussianNoise> -->
+        <jointName>hex_sensor_joint</jointName>
+    </plugin>
+  </gazebo>
 </robot>
